Commit message: renamed from rplidar to laser_sensor

File: turtlebot4_description/urdf/sensors/rplidar.urdf.xacro (robot description, xacro)
@@ -1,5 +1,5 @@
 <?xml version="1.0"?>
 <robot xmlns:xacro="http://ros.org/wiki/xacro">
-<xacro:macro name="rplidar" params="name parent_link gazebo *origin">
+<xacro:macro name="laser_sensor" params="name parent_link gazebo *origin">
   <xacro:include filename="$(find irobot_create_description)/urdf/common_properties.urdf.xacro"/>
   <xacro:property name="mass"       value="0.17"/>
